Commit message: Set URDF joint effort limits to rated torques

File: urdf/orion5.urdf (robot description, URDF)
Before this commit: robot orion5, 9 links, 8 joints
Joints:
- joint joint_1: limit lower=-3.14 upper=3.14 effort=200 velocity=1.57 -> lower=-3.14 upper=3.14 effort=87 velocity=1.57
- joint joint_2: limit lower=-3.14 upper=3.14 effort=200 velocity=1.57 -> lower=-3.14 upper=3.14 effort=87 velocity=1.57
- joint joint_3: limit lower=-3.14 upper=3.14 effort=200 velocity=1.57 -> lower=-3.14 upper=3.14 effort=52 velocity=1.57
- joint joint_4: limit lower=-3.14 upper=3.14 effort=200 velocity=1.57 -> lower=-3.14 upper=3.14 effort=10 velocity=1.57
- joint joint_5: limit lower=-3.14 upper=3.14 effort=200 velocity=1.57 -> lower=-3.14 upper=3.14 effort=10 velocity=1.57
- joint joint_6: limit lower=-3.14 upper=3.14 effort=200 velocity=1.57 -> lower=-3.14 upper=3.14 effort=10 velocity=1.57
